File: controller.sch (KiCad schematic (older format))
At the start: 12 parts

Commit message: Annotate and add negative IOC faults.
Parts:
- gave numbers to parts that had none: 12
Changed lines of the file:
@@
 $EndDescr
 $Comp
-L PIC32MK1024MCF064 U?
+L PIC32MK1024MCF064 U1
 U 1 1 5AEC26E4
 P 6550 3800
-F 0 "U?" H 6550 2100 60  0000 C CNN
+F 0 "U1" H 6550 2100 60  0000 C CNN
 F 1 "PIC32MK1024MCF064" H 6600 5450 60  0000 C CNN
 F 2 "" H 5850 3800 60  0001 C CNN
@@
 $EndComp
 $Comp
-L Crystal Y?
+L Crystal Y1
 U 1 1 5AEC26EB
 P 9900 4550
-F 0 "Y?" H 9900 4700 50  0000 C CNN
+F 0 "Y1" H 9900 4700 50  0000 C CNN
 F 1 "12MHz" H 9900 4400 50  0000 C CNN
 F 2 "" H 9900 4550 50  0001 C CNN
@@
 $EndComp
 $Comp
-L C C?
+L C C7
 U 1 1 5AEC26F2
 P 10100 4350
-F 0 "C?" H 10125 4450 50  0000 L CNN
+F 0 "C7" H 10125 4450 50  0000 L CNN
 F 1 "8p" H 10125 4250 50  0000 L CNN
 F 2 "" H 10138 4200 50  0001 C CNN
@@
 $EndComp
 $Comp
-L C C?
+L C C8
 U 1 1 5AEC26F9
 P 10100 4750
-F 0 "C?" H 10125 4850 50  0000 L CNN
+F 0 "C8" H 10125 4850 50  0000 L CNN
 F 1 "8p" H 10125 4650 50  0000 L CNN
 F 2 "" H 10138 4600 50  0001 C CNN
@@
 $EndComp
 $Comp
-L R R?
+L R R2
 U 1 1 5AEC2700
 P 9700 4350
-F 0 "R?" V 9780 4350 50  0000 C CNN
+F 0 "R2" V 9780 4350 50  0000 C CNN
 F 1 "1k" V 9700 4350 50  0000 C CNN
 F 2 "" V 9630 4350 50  0001 C CNN
@@
 $EndComp
 $Comp
-L GND #PWR01
+L GND #PWR15
 U 1 1 5AEC2707
 P 10300 4550
-F 0 "#PWR01" H 10300 4300 50  0001 C CNN
+F 0 "#PWR15" H 10300 4300 50  0001 C CNN
 F 1 "GND" H 10300 4400 50  0000 C CNN
 F 2 "" H 10300 4550 50  0001 C CNN
@@
 $EndComp
 $Comp
-L GND #PWR02
+L GND #PWR4
 U 1 1 5AEC270D
 P 3550 3050
-F 0 "#PWR02" H 3550 2800 50  0001 C CNN
+F 0 "#PWR4" H 3550 2800 50  0001 C CNN
 F 1 "GND" H 3550 2900 50  0000 C CNN
 F 2 "" H 3550 3050 50  0001 C CNN
@@
 $EndComp
 $Comp
-L C C?
+L C C2
 U 1 1 5AEC2713
 P 3700 3150
-F 0 "C?" H 3725 3250 50  0000 L CNN
+F 0 "C2" H 3725 3250 50  0000 L CNN
 F 1 "0.1u" H 3725 3050 50  0000 L CNN
 F 2 "" H 3738 3000 50  0001 C CNN
@@
 $EndComp
 $Comp
-L +5V #PWR03
+L +5V #PWR5
 U 1 1 5AEC271A
 P 3550 3250
-F 0 "#PWR03" H 3550 3100 50  0001 C CNN
+F 0 "#PWR5" H 3550 3100 50  0001 C CNN
 F 1 "+5V" H 3550 3390 50  0000 C CNN
 F 2 "" H 3550 3250 50  0001 C CNN
@@
 $EndComp
 $Comp
-L GND #PWR04
+L GND #PWR8
 U 1 1 5AEC2720
 P 3550 4650
-F 0 "#PWR04" H 3550 4400 50  0001 C CNN
+F 0 "#PWR8" H 3550 4400 50  0001 C CNN
 F 1 "GND" H 3550 4500 50  0000 C CNN
 F 2 "" H 3550 4650 50  0001 C CNN
@@
 $EndComp
 $Comp
-L C C?
+L C C4
 U 1 1 5AEC2726
 P 3700 4750
-F 0 "C?" H 3725 4850 50  0000 L CNN
+F 0 "C4" H 3725 4850 50  0000 L CNN
 F 1 "0.1u" H 3725 4650 50  0000 L CNN
 F 2 "" H 3738 4600 50  0001 C CNN
@@
 $EndComp
 $Comp
-L +5V #PWR05
+L +5V #PWR9
 U 1 1 5AEC272D
 P 3550 4850
-F 0 "#PWR05" H 3550 4700 50  0001 C CNN
+F 0 "#PWR9" H 3550 4700 50  0001 C CNN
 F 1 "+5V" H 3550 4990 50  0000 C CNN
 F 2 "" H 3550 4850 50  0001 C CNN
@@
 $EndComp
 $Comp
-L GND #PWR06
+L GND #PWR13
 U 1 1 5AEC2733
 P 9700 3050
-F 0 "#PWR06" H 9700 2800 50  0001 C CNN
+F 0 "#PWR13" H 9700 2800 50  0001 C CNN
 F 1 "GND" H 9700 2900 50  0000 C CNN
 F 2 "" H 9700 3050 50  0001 C CNN
@@
 $EndComp
 $Comp
-L C C?
+L C C5
 U 1 1 5AEC2739
 P 9550 2950
-F 0 "C?" H 9575 3050 50  0000 L CNN
+F 0 "C5" H 9575 3050 50  0000 L CNN
 F 1 "0.1u" H 9575 2850 50  0000 L CNN
 F 2 "" H 9588 2800 50  0001 C CNN
@@
 $EndComp
 $Comp
-L +5V #PWR07
+L +5V #PWR12
 U 1 1 5AEC2740
 P 9700 2850
-F 0 "#PWR07" H 9700 2700 50  0001 C CNN
+F 0 "#PWR12" H 9700 2700 50  0001 C CNN
 F 1 "+5V" H 9700 2990 50  0000 C CNN
 F 2 "" H 9700 2850 50  0001 C CNN
@@
 $EndComp
 $Comp
-L GND #PWR08
+L GND #PWR7
 U 1 1 5AEC2746
 P 3550 4150
-F 0 "#PWR08" H 3550 3900 50  0001 C CNN
+F 0 "#PWR7" H 3550 3900 50  0001 C CNN
 F 1 "GND" H 3550 4000 50  0000 C CNN
 F 2 "" H 3550 4150 50  0001 C CNN
@@
 $EndComp
 $Comp
-L C C?
+L C C3
 U 1 1 5AEC274C
 P 3700 4050
-F 0 "C?" H 3725 4150 50  0000 L CNN
+F 0 "C3" H 3725 4150 50  0000 L CNN
 F 1 "0.1u" H 3725 3950 50  0000 L CNN
 F 2 "" H 3738 3900 50  0001 C CNN
@@
 $EndComp
 $Comp
-L +5V #PWR09
+L +5V #PWR6
 U 1 1 5AEC2753
 P 3550 3950
-F 0 "#PWR09" H 3550 3800 50  0001 C CNN
+F 0 "#PWR6" H 3550 3800 50  0001 C CNN
 F 1 "+5V" H 3550 4090 50  0000 C CNN
 F 2 "" H 3550 3950 50  0001 C CNN
@@
 $EndComp
 $Comp
-L GND #PWR010
+L GND #PWR10
 U 1 1 5AEC2759
 P 9350 4550
-F 0 "#PWR010" H 9350 4300 50  0001 C CNN
+F 0 "#PWR10" H 9350 4300 50  0001 C CNN
 F 1 "GND" H 9350 4400 50  0000 C CNN
 F 2 "" H 9350 4550 50  0001 C CNN
@@
 $EndComp
 $Comp
-L GND #PWR011
+L GND #PWR14
 U 1 1 5AEC275F
 P 9900 5000
-F 0 "#PWR011" H 9900 4750 50  0001 C CNN
+F 0 "#PWR14" H 9900 4750 50  0001 C CNN
 F 1 "GND" H 9900 4850 50  0000 C CNN
 F 2 "" H 9900 5000 50  0001 C CNN
@@
 $EndComp
 $Comp
-L C C?
+L C C6
 U 1 1 5AEC2765
 P 9700 5000
-F 0 "C?" H 9725 5100 50  0000 L CNN
+F 0 "C6" H 9725 5100 50  0000 L CNN
 F 1 "0.1u" H 9725 4900 50  0000 L CNN
 F 2 "" H 9738 4850 50  0001 C CNN
@@
 $EndComp
 $Comp
-L +5V #PWR012
+L +5V #PWR11
 U 1 1 5AEC276C
 P 9400 4850
-F 0 "#PWR012" H 9400 4700 50  0001 C CNN
+F 0 "#PWR11" H 9400 4700 50  0001 C CNN
 F 1 "+5V" H 9400 4990 50  0000 C CNN
 F 2 "" H 9400 4850 50  0001 C CNN
@@
 $EndComp
 $Comp
-L R R?
+L R R1
 U 1 1 5AEC2772
 P 1350 1750
-F 0 "R?" V 1430 1750 50  0000 C CNN
+F 0 "R1" V 1430 1750 50  0000 C CNN
 F 1 "10k" V 1350 1750 50  0000 C CNN
 F 2 "" V 1280 1750 50  0001 C CNN
@@
 $EndComp
 $Comp
-L C C?
+L C C1
 U 1 1 5AEC2779
 P 1350 2150
-F 0 "C?" H 1375 2250 50  0000 L CNN
+F 0 "C1" H 1375 2250 50  0000 L CNN
 F 1 "0.1u" H 1375 2050 50  0000 L CNN
 F 2 "" H 1388 2000 50  0001 C CNN
@@
 $EndComp
 $Comp
-L GND #PWR013
+L GND #PWR2
 U 1 1 5AEC2780
 P 1350 2350
-F 0 "#PWR013" H 1350 2100 50  0001 C CNN
+F 0 "#PWR2" H 1350 2100 50  0001 C CNN
 F 1 "GND" H 1350 2200 50  0000 C CNN
 F 2 "" H 1350 2350 50  0001 C CNN
@@
 $EndComp
 $Comp
-L +5V #PWR014
+L +5V #PWR1
 U 1 1 5AEC2786
 P 1350 1550
-F 0 "#PWR014" H 1350 1400 50  0001 C CNN
+F 0 "#PWR1" H 1350 1400 50  0001 C CNN
 F 1 "+5V" H 1350 1690 50  0000 C CNN
 F 2 "" H 1350 1550 50  0001 C CNN
@@
 INDX1
 $Comp
-L GND #PWR?
+L GND #PWR3
 U 1 1 5AEFD8E9
 P 3350 3650
-F 0 "#PWR?" H 3350 3400 50  0001 C CNN
+F 0 "#PWR3" H 3350 3400 50  0001 C CNN
 F 1 "GND" H 3350 3500 50  0000 C CNN
 F 2 "" H 3350 3650 50  0001 C CNN
