File: desat.sch (KiCad schematic (older format))
At the start: 8 parts

Commit message: Annotate and add negative IOC faults.
Parts:
- gave numbers to parts that had none: 2
Changed lines of the file:
@@
 $EndDescr
 $Comp
-L 7400 U?
+L 7400 U2
 U 1 1 5AF0C78B
 P 5000 2250
-F 0 "U?" H 5000 2300 50  0000 C CNN
+F 0 "U2" H 5000 2300 50  0000 C CNN
 F 1 "7400" H 5000 2150 50  0000 C CNN
 F 2 "" H 5000 2250 50  0001 C CNN
@@
 $EndComp
 $Comp
-L 7400 U?
+L 7400 U2
 U 2 1 5AF0C7D2
 P 5000 2850
-F 0 "U?" H 5000 2900 50  0000 C CNN
+F 0 "U2" H 5000 2900 50  0000 C CNN
 F 1 "7400" H 5000 2750 50  0000 C CNN
 F 2 "" H 5000 2850 50  0001 C CNN
@@
 $EndComp
 $Comp
-L 7400 U?
+L 7400 U2
 U 3 1 5AF0C823
 P 5000 3450
-F 0 "U?" H 5000 3500 50  0000 C CNN
+F 0 "U2" H 5000 3500 50  0000 C CNN
 F 1 "7400" H 5000 3350 50  0000 C CNN
 F 2 "" H 5000 3450 50  0001 C CNN
@@
 $EndComp
 $Comp
-L 7400 U?
+L 7400 U2
 U 4 1 5AF0C880
 P 5000 4050
-F 0 "U?" H 5000 4100 50  0000 C CNN
+F 0 "U2" H 5000 4100 50  0000 C CNN
 F 1 "7400" H 5000 3950 50  0000 C CNN
 F 2 "" H 5000 4050 50  0001 C CNN
@@
 DESAT_C-
 $Comp
-L 74LS32 U?
+L 74LS32 U3
 U 1 1 5AF0CC82
 P 6450 2550
-F 0 "U?" H 6450 2600 50  0000 C CNN
+F 0 "U3" H 6450 2600 50  0000 C CNN
 F 1 "74LS32" H 6450 2500 50  0000 C CNN
 F 2 "" H 6450 2550 50  0001 C CNN
@@
 $EndComp
 $Comp
-L 74LS32 U?
+L 74LS32 U3
 U 2 1 5AF0CCE3
 P 6450 3150
-F 0 "U?" H 6450 3200 50  0000 C CNN
+F 0 "U3" H 6450 3200 50  0000 C CNN
 F 1 "74LS32" H 6450 3100 50  0000 C CNN
 F 2 "" H 6450 3150 50  0001 C CNN
@@
 $EndComp
 $Comp
-L 74LS32 U?
+L 74LS32 U3
 U 3 1 5AF0CE3A
 P 6450 3750
-F 0 "U?" H 6450 3800 50  0000 C CNN
+F 0 "U3" H 6450 3800 50  0000 C CNN
 F 1 "74LS32" H 6450 3700 50  0000 C CNN
 F 2 "" H 6450 3750 50  0001 C CNN
@@
 $EndComp
 $Comp
-L 74LS32 U?
+L 74LS32 U3
 U 4 1 5AF0CE7B
 P 6450 4350
-F 0 "U?" H 6450 4400 50  0000 C CNN
+F 0 "U3" H 6450 4400 50  0000 C CNN
 F 1 "74LS32" H 6450 4300 50  0000 C CNN
 F 2 "" H 6450 4350 50  0001 C CNN
