File: motor_current.sch (KiCad schematic (older format))
At the start: 6 parts, among them J5 I_A, J6 I_B, J7 I_C

Commit message: Adds IOC reference points.
Connections:
- net I_A_0REF: now reaches J5.4 (Pin_4)
- net I_B_0REF: now reaches J6.4 (Pin_4)
- net I_C_0REF: now reaches J7.4 (Pin_4)
Other:
- note added: "Current Sensor Connectors\n\nAssuming Current Transducer with:\n2.5V + k*I/In Behavior"
- note removed: "Current Sensor Connectors\n\nAssuming Current Transducer with:\n2.5V + k*I/In Behavior\n\n4th Pin is Vref, which is assumed\nstatic in this design"
Changed lines of the file:
@@
 $Descr A4 11693 8268
 encoding utf-8
-Sheet 7 19
+Sheet 19 19
 Title ""
 Date ""
@@
 $EndComp
 Text Notes 1700 1900 0    60   ~ 0
-Current Sensor Connectors\n\nAssuming Current Transducer with:\n2.5V + k*I/In Behavior\n\n4th Pin is Vref, which is assumed\nstatic in this design
+Current Sensor Connectors\n\nAssuming Current Transducer with:\n2.5V + k*I/In Behavior
 $Comp
 L R R5
@@
 Text HLabel 2450 3400 2    60   Input ~ 0
 I_C_SENSE
+Text HLabel 2450 2500 2    60   Input ~ 0
+I_A_0REF
+Wire Wire Line
+	2450 2500 2050 2500
+Wire Wire Line
+	2050 2500 2050 2400
+Text HLabel 2450 3150 2    60   Input ~ 0
+I_B_0REF
+Wire Wire Line
+	2450 3150 2050 3150
+Wire Wire Line
+	2050 3150 2050 3050
+Text HLabel 2450 3800 2    60   Input ~ 0
+I_C_0REF
+Wire Wire Line
+	2450 3800 2050 3800
+Wire Wire Line
+	2050 3800 2050 3700
 $EndSCHEMATC
