File: motor_current.sch (KiCad schematic (older format))
At the start: 6 parts

Commit message: Annotate and add negative IOC faults.
Parts:
- gave numbers to parts that had none: 6
Changed lines of the file:
@@
 $EndDescr
 $Comp
-L GND #PWR029
+L GND #PWR31
 U 1 1 5AEC79CD
 P 2450 2300
-F 0 "#PWR029" H 2450 2050 50  0001 C CNN
+F 0 "#PWR31" H 2450 2050 50  0001 C CNN
 F 1 "GND" H 2450 2150 50  0000 C CNN
 F 2 "" H 2450 2300 50  0001 C CNN
@@
 $EndComp
 $Comp
-L +5V #PWR030
+L +5V #PWR30
 U 1 1 5AEC79D3
 P 2450 2200
-F 0 "#PWR030" H 2450 2050 50  0001 C CNN
+F 0 "#PWR30" H 2450 2050 50  0001 C CNN
 F 1 "+5V" H 2450 2340 50  0000 C CNN
 F 2 "" H 2450 2200 50  0001 C CNN
@@
 Current Sensor Connectors\n\nAssuming Current Transducer with:\n2.5V + k*I/In Behavior\n\n4th Pin is Vref, which is assumed\nstatic in this design
 $Comp
-L R R?
+L R R5
 U 1 1 5AEC79DA
 P 2250 2400
-F 0 "R?" V 2330 2400 50  0000 C CNN
+F 0 "R5" V 2330 2400 50  0000 C CNN
 F 1 "10k" V 2250 2400 50  0000 C CNN
 F 2 "" V 2180 2400 50  0001 C CNN
@@
 $EndComp
 $Comp
-L GND #PWR031
+L GND #PWR33
 U 1 1 5AEC79E2
 P 2450 2950
-F 0 "#PWR031" H 2450 2700 50  0001 C CNN
+F 0 "#PWR33" H 2450 2700 50  0001 C CNN
 F 1 "GND" H 2450 2800 50  0000 C CNN
 F 2 "" H 2450 2950 50  0001 C CNN
@@
 $EndComp
 $Comp
-L +5V #PWR032
+L +5V #PWR32
 U 1 1 5AEC79E8
 P 2450 2850
-F 0 "#PWR032" H 2450 2700 50  0001 C CNN
+F 0 "#PWR32" H 2450 2700 50  0001 C CNN
 F 1 "+5V" H 2450 2990 50  0000 C CNN
 F 2 "" H 2450 2850 50  0001 C CNN
@@
 $EndComp
 $Comp
-L R R?
+L R R6
 U 1 1 5AEC79EE
 P 2250 3050
-F 0 "R?" V 2330 3050 50  0000 C CNN
+F 0 "R6" V 2330 3050 50  0000 C CNN
 F 1 "10k" V 2250 3050 50  0000 C CNN
 F 2 "" V 2180 3050 50  0001 C CNN
@@
 $EndComp
 $Comp
-L GND #PWR033
+L GND #PWR35
 U 1 1 5AEC79F6
 P 2450 3600
-F 0 "#PWR033" H 2450 3350 50  0001 C CNN
+F 0 "#PWR35" H 2450 3350 50  0001 C CNN
 F 1 "GND" H 2450 3450 50  0000 C CNN
 F 2 "" H 2450 3600 50  0001 C CNN
@@
 $EndComp
 $Comp
-L +5V #PWR034
+L +5V #PWR34
 U 1 1 5AEC79FC
 P 2450 3500
-F 0 "#PWR034" H 2450 3350 50  0001 C CNN
+F 0 "#PWR34" H 2450 3350 50  0001 C CNN
 F 1 "+5V" H 2450 3640 50  0000 C CNN
 F 2 "" H 2450 3500 50  0001 C CNN
@@
 $EndComp
 $Comp
-L R R?
+L R R7
 U 1 1 5AEC7A02
 P 2250 3700
-F 0 "R?" V 2330 3700 50  0000 C CNN
+F 0 "R7" V 2330 3700 50  0000 C CNN
 F 1 "10k" V 2250 3700 50  0000 C CNN
 F 2 "" V 2180 3700 50  0001 C CNN
@@
 	2450 3700 2450 3600
 $Comp
-L Conn_01x04 J?
+L Conn_01x04 J5
 U 1 1 5AEC7A85
 P 1850 2200
-F 0 "J?" H 1850 2400 50  0000 C CNN
+F 0 "J5" H 1850 2400 50  0000 C CNN
 F 1 "I_A" H 1850 1900 50  0000 C CNN
 F 2 "" H 1850 2200 50  0001 C CNN
@@
 $EndComp
 $Comp
-L Conn_01x04 J?
+L Conn_01x04 J6
 U 1 1 5AEC7A8D
 P 1850 2850
-F 0 "J?" H 1850 3050 50  0000 C CNN
+F 0 "J6" H 1850 3050 50  0000 C CNN
 F 1 "I_B" H 1850 2550 50  0000 C CNN
 F 2 "" H 1850 2850 50  0001 C CNN
@@
 $EndComp
 $Comp
-L Conn_01x04 J?
+L Conn_01x04 J7
 U 1 1 5AEC7A94
 P 1850 3500
-F 0 "J?" H 1850 3700 50  0000 C CNN
+F 0 "J7" H 1850 3700 50  0000 C CNN
 F 1 "I_C" H 1850 3200 50  0000 C CNN
 F 2 "" H 1850 3500 50  0001 C CNN
