File: current_faults.sch (KiCad schematic (older format))
At the start: 8 parts

Commit message: Implement temperature sensor amplifier.
Other:
- note added: "TODO(willjschmitt): Set negative direction IOC."
Changed lines of the file:
@@
 $Descr A4 11693 8268
 encoding utf-8
-Sheet 11 18
+Sheet 11 19
 Title ""
 Date ""
@@
 Text Notes 850  950  0    60   ~ 0
 TODO(willjschmitt): Set IOC_REF to reasonable value.
+Text Notes 850  800  0    60   ~ 0
+TODO(willjschmitt): Set negative direction IOC.
 $EndSCHEMATC

Commit message: Annotate and add negative IOC faults.
Parts:
- added U? (x2): LMV393, symbol LMV393
- added U? (x2): 74LS32, symbol 74LS32
- gave numbers to parts that had none: 3
Connections:
- net +5V: now also U?.8 (V+), U?.8 (V+)
- net GND: now also U?.4 (V-), U?.4 (V-), U?.7 (GND), U?.7 (GND)
- net IOC_FAULT: now also U?.6; no longer U6.6
- net I_A: now also U4.2 (_), U4.5 (+); no longer U4.3 (+)
- net I_B: now also U5.2 (_), U5.5 (+); no longer U4.5 (+)
- net I_C: now also U?.2 (_), U?.3 (+); no longer U5.3 (+)
- net VCC: now also U?.14 (VCC), U?.14 (VCC)
- net at U5.1: now also U6.4; no longer U6.5
- net +IOC_REF: now reaches U5.6 (_)
- net +IOC_REF: now also U4.6 (_), U?.2 (_)
- net at U5.7: now also U6.5
- net at U6.3: now also U?.1; no longer U6.4
- net at U6.10: now also U?.1
- net at U6.8: now also U?.5
- net at U6.9: now also U?.1
- removed net IOC_REF: U4.2 (_), U4.6 (_), U5.2 (_)
- new net: U6.6, U?.2
- new net: U?.3, U?.4
- new net -IOC_REF: U4.3 (+), U5.3 (+), U?.3 (+)
Other:
- moved on the sheet: U6B, U6C, U6D

Commit message: Deduping kty_84 sheet names.
Parts:
- gave numbers to parts that had none: 2
Connections:
- net +IOC_REF: now also U14.6 (_); no longer U14.2 (_)
- net I_C: now also U14.5 (+); no longer U14.3 (+)
- net at U6.10: now also U14.7; no longer U14.1
Changed lines of the file:
@@
 $EndComp
 $Comp
-L GND #PWR43
+L GND #PWR040
 U 1 1 5AF2611D
 P 2100 2800
-F 0 "#PWR43" H 2100 2550 50  0001 C CNN
+F 0 "#PWR040" H 2100 2550 50  0001 C CNN
 F 1 "GND" H 2100 2650 50  0000 C CNN
 F 2 "" H 2100 2800 50  0001 C CNN
@@
 $EndComp
 $Comp
-L GND #PWR41
+L GND #PWR041
 U 1 1 5AF26150
 P 2100 1800
-F 0 "#PWR41" H 2100 1550 50  0001 C CNN
+F 0 "#PWR041" H 2100 1550 50  0001 C CNN
 F 1 "GND" H 2100 1650 50  0000 C CNN
 F 2 "" H 2100 1800 50  0001 C CNN
@@
 $EndComp
 $Comp
-L GND #PWR45
+L GND #PWR042
 U 1 1 5AF261AC
 P 2100 3800
-F 0 "#PWR45" H 2100 3550 50  0001 C CNN
+F 0 "#PWR042" H 2100 3550 50  0001 C CNN
 F 1 "GND" H 2100 3650 50  0000 C CNN
 F 2 "" H 2100 3800 50  0001 C CNN
@@
 $EndComp
 $Comp
-L GND #PWR47
+L GND #PWR043
 U 1 1 5AF261C8
 P 2100 4800
-F 0 "#PWR47" H 2100 4550 50  0001 C CNN
+F 0 "#PWR043" H 2100 4550 50  0001 C CNN
 F 1 "GND" H 2100 4650 50  0000 C CNN
 F 2 "" H 2100 4800 50  0001 C CNN
@@
 $EndComp
 $Comp
-L +5V #PWR40
+L +5V #PWR044
 U 1 1 5AF26F2F
 P 2100 1200
-F 0 "#PWR40" H 2100 1050 50  0001 C CNN
+F 0 "#PWR044" H 2100 1050 50  0001 C CNN
 F 1 "+5V" H 2100 1340 50  0000 C CNN
 F 2 "" H 2100 1200 50  0001 C CNN
@@
 $EndComp
 $Comp
-L +5V #PWR42
+L +5V #PWR045
 U 1 1 5AF27223
 P 2100 2200
-F 0 "#PWR42" H 2100 2050 50  0001 C CNN
+F 0 "#PWR045" H 2100 2050 50  0001 C CNN
 F 1 "+5V" H 2100 2340 50  0000 C CNN
 F 2 "" H 2100 2200 50  0001 C CNN
@@
 $EndComp
 $Comp
-L +5V #PWR44
+L +5V #PWR046
 U 1 1 5AF2736E
 P 2100 3200
-F 0 "#PWR44" H 2100 3050 50  0001 C CNN
+F 0 "#PWR046" H 2100 3050 50  0001 C CNN
 F 1 "+5V" H 2100 3340 50  0000 C CNN
 F 2 "" H 2100 3200 50  0001 C CNN
@@
 $EndComp
 $Comp
-L +5V #PWR46
+L +5V #PWR047
 U 1 1 5AF27419
 P 2100 4200
-F 0 "#PWR46" H 2100 4050 50  0001 C CNN
+F 0 "#PWR047" H 2100 4050 50  0001 C CNN
 F 1 "+5V" H 2100 4340 50  0000 C CNN
 F 2 "" H 2100 4200 50  0001 C CNN
@@
 I_C
 $Comp
-L LMV393 U?
+L LMV393 U14
 U 1 1 5AF08203
 P 2200 5500
-F 0 "U?" H 2350 5650 50  0000 C CNN
+F 0 "U14" H 2350 5650 50  0000 C CNN
 F 1 "LMV393" H 2450 5350 50  0000 C CNN
 F 2 "" H 2200 5500 50  0001 C CNN
@@
 $EndComp
 $Comp
-L LMV393 U?
-U 1 1 5AF0820A
+L LMV393 U14
+U 2 1 5AF0820A
 P 2200 6500
-F 0 "U?" H 2350 6650 50  0000 C CNN
+F 0 "U14" H 2350 6650 50  0000 C CNN
 F 1 "LMV393" H 2450 6350 50  0000 C CNN
 F 2 "" H 2200 6500 50  0001 C CNN
 F 3 "" H 2200 6500 50  0001 C CNN
-	1    2200 6500
-	1    0    0    -1
-$EndComp
-$Comp
-L GND #PWR?
+	2    2200 6500
+	1    0    0    -1
+$EndComp
+$Comp
+L GND #PWR048
 U 1 1 5AF08211
 P 2100 5800
-F 0 "#PWR?" H 2100 5550 50  0001 C CNN
+F 0 "#PWR048" H 2100 5550 50  0001 C CNN
 F 1 "GND" H 2100 5650 50  0000 C CNN
 F 2 "" H 2100 5800 50  0001 C CNN
@@
 $EndComp
 $Comp
-L GND #PWR?
+L GND #PWR049
 U 1 1 5AF08217
 P 2100 6800
-F 0 "#PWR?" H 2100 6550 50  0001 C CNN
+F 0 "#PWR049" H 2100 6550 50  0001 C CNN
 F 1 "GND" H 2100 6650 50  0000 C CNN
 F 2 "" H 2100 6800 50  0001 C CNN
@@
 	1700 5600 1900 5600
 $Comp
-L +5V #PWR?
+L +5V #PWR050
 U 1 1 5AF08220
 P 2100 5200
-F 0 "#PWR?" H 2100 5050 50  0001 C CNN
+F 0 "#PWR050" H 2100 5050 50  0001 C CNN
 F 1 "+5V" H 2100 5340 50  0000 C CNN
 F 2 "" H 2100 5200 50  0001 C CNN
@@
 $EndComp
 $Comp
-L +5V #PWR?
+L +5V #PWR051
 U 1 1 5AF08226
 P 2100 6200
-F 0 "#PWR?" H 2100 6050 50  0001 C CNN
+F 0 "#PWR051" H 2100 6050 50  0001 C CNN
 F 1 "+5V" H 2100 6340 50  0000 C CNN
 F 2 "" H 2100 6200 50  0001 C CNN
@@
 	6250 5000 6150 5000
 $Comp
-L 74LS32 U?
+L 74LS32 U15
 U 1 1 5AF08CE3
 P 5550 3050
-F 0 "U?" H 5550 3100 50  0000 C CNN
+F 0 "U15" H 5550 3100 50  0000 C CNN
 F 1 "74LS32" H 5550 3000 50  0000 C CNN
 F 2 "" H 5550 3050 50  0001 C CNN
@@
 $EndComp
 $Comp
-L 74LS32 U?
+L 74LS32 U15
 U 2 1 5AF08D1E
 P 5550 5000
-F 0 "U?" H 5550 5050 50  0000 C CNN
+F 0 "U15" H 5550 5050 50  0000 C CNN
 F 1 "74LS32" H 5550 4950 50  0000 C CNN
 F 2 "" H 5550 5000 50  0001 C CNN
