File: igbt.sch (KiCad schematic (older format))
At the start: 1 part

Commit message: Annotate and add negative IOC faults.
Parts:
- gave numbers to parts that had none: 1
Changed lines of the file:
@@
 $EndDescr
 $Comp
-L Conn_01x09 J?
+L Conn_01x09 J1
 U 1 1 5AED5E26
 P 2050 1750
-AR Path="/5AED5DDF/5AED5E26" Ref="J?"  Part="1"
-AR Path="/5AEDA321/5AED5E26" Ref="J?"  Part="1"
-AR Path="/5AEDAF6D/5AED5E26" Ref="J?"  Part="1"
-F 0 "J?" H 2050 2250 50  0000 C CNN
+AR Path="/5AED5DDF/5AED5E26" Ref="J1"  Part="1"
+AR Path="/5AEDA321/5AED5E26" Ref="J2"  Part="1"
+AR Path="/5AEDAF6D/5AED5E26" Ref="J3"  Part="1"
+F 0 "J3" H 2050 2250 50  0000 C CNN
 F 1 "IGBT" H 2050 1250 50  0000 C CNN
 F 2 "" H 2050 1750 50  0001 C CNN
@@
 $EndComp
 $Comp
-L GND #PWR015
+L GND #PWR16
 U 1 1 5AED6001
 P 1650 1350
-AR Path="/5AED5DDF/5AED6001" Ref="#PWR015"  Part="1"
-AR Path="/5AEDA321/5AED6001" Ref="#PWR018"  Part="1"
-AR Path="/5AEDAF6D/5AED6001" Ref="#PWR021"  Part="1"
-F 0 "#PWR015" H 1650 1100 50  0001 C CNN
+AR Path="/5AED5DDF/5AED6001" Ref="#PWR16"  Part="1"
+AR Path="/5AEDA321/5AED6001" Ref="#PWR19"  Part="1"
+AR Path="/5AEDAF6D/5AED6001" Ref="#PWR22"  Part="1"
+F 0 "#PWR22" H 1650 1100 50  0001 C CNN
 F 1 "GND" H 1650 1200 50  0000 C CNN
 F 2 "" H 1650 1350 50  0001 C CNN
@@
 $EndComp
 $Comp
-L +5V #PWR016
+L +5V #PWR17
 U 1 1 5AED6017
 P 1650 1450
-AR Path="/5AED5DDF/5AED6017" Ref="#PWR016"  Part="1"
-AR Path="/5AEDA321/5AED6017" Ref="#PWR019"  Part="1"
-AR Path="/5AEDAF6D/5AED6017" Ref="#PWR022"  Part="1"
-F 0 "#PWR016" H 1650 1300 50  0001 C CNN
+AR Path="/5AED5DDF/5AED6017" Ref="#PWR17"  Part="1"
+AR Path="/5AEDA321/5AED6017" Ref="#PWR20"  Part="1"
+AR Path="/5AEDAF6D/5AED6017" Ref="#PWR23"  Part="1"
+F 0 "#PWR23" H 1650 1300 50  0001 C CNN
 F 1 "+5V" H 1650 1590 50  0000 C CNN
 F 2 "" H 1650 1450 50  0001 C CNN
@@
 $EndComp
 $Comp
-L +24V #PWR017
+L +24V #PWR18
 U 1 1 5AED602D
 P 1650 1550
-AR Path="/5AED5DDF/5AED602D" Ref="#PWR017"  Part="1"
-AR Path="/5AEDA321/5AED602D" Ref="#PWR020"  Part="1"
-AR Path="/5AEDAF6D/5AED602D" Ref="#PWR023"  Part="1"
-F 0 "#PWR017" H 1650 1400 50  0001 C CNN
+AR Path="/5AED5DDF/5AED602D" Ref="#PWR18"  Part="1"
+AR Path="/5AEDA321/5AED602D" Ref="#PWR21"  Part="1"
+AR Path="/5AEDAF6D/5AED602D" Ref="#PWR24"  Part="1"
+F 0 "#PWR24" H 1650 1400 50  0001 C CNN
 F 1 "+24V" H 1650 1690 50  0000 C CNN
 F 2 "" H 1650 1550 50  0001 C CNN
