File: motor.sch (KiCad schematic (older format))
At the start: 3 parts

Commit message: Annotate and add negative IOC faults.
Parts:
- gave numbers to parts that had none: 3
Changed lines of the file:
@@
 $EndDescr
 $Comp
-L Conn_01x12 J?
+L Conn_01x12 J4
 U 1 1 5AEDE476
 P 1450 2050
-F 0 "J?" H 1450 2650 50  0000 C CNN
+F 0 "J4" H 1450 2650 50  0000 C CNN
 F 1 "MOTOR_ENCODER" H 1450 1350 50  0000 C CNN
 F 2 "" H 1450 2050 50  0001 C CNN
@@
 $EndComp
 $Comp
-L +5V #PWR024
+L +5V #PWR25
 U 1 1 5AEDE47D
 P 1750 1850
-F 0 "#PWR024" H 1750 1700 50  0001 C CNN
+F 0 "#PWR25" H 1750 1700 50  0001 C CNN
 F 1 "+5V" H 1750 1990 50  0000 C CNN
 F 2 "" H 1750 1850 50  0001 C CNN
@@
 $EndComp
 $Comp
-L GND #PWR025
+L GND #PWR26
 U 1 1 5AEDE483
 P 1750 1950
-F 0 "#PWR025" H 1750 1700 50  0001 C CNN
+F 0 "#PWR26" H 1750 1700 50  0001 C CNN
 F 1 "GND" H 1750 1800 50  0000 C CNN
 F 2 "" H 1750 1950 50  0001 C CNN
@@
 $EndComp
 $Comp
-L R R?
+L R R3
 U 1 1 5AEDE489
 P 2050 2150
-F 0 "R?" V 2130 2150 50  0000 C CNN
+F 0 "R3" V 2130 2150 50  0000 C CNN
 F 1 "2k" V 2050 2150 50  0000 C CNN
 F 2 "" V 1980 2150 50  0001 C CNN
@@
 $EndComp
 $Comp
-L R R?
+L R R4
 U 1 1 5AEDE490
 P 2050 2750
-F 0 "R?" V 2130 2750 50  0000 C CNN
+F 0 "R4" V 2130 2750 50  0000 C CNN
 F 1 "2k" V 2050 2750 50  0000 C CNN
 F 2 "" V 1980 2750 50  0001 C CNN
@@
 $EndComp
 $Comp
-L GND #PWR026
+L GND #PWR29
 U 1 1 5AEDE497
 P 2350 2600
-F 0 "#PWR026" H 2350 2350 50  0001 C CNN
+F 0 "#PWR29" H 2350 2350 50  0001 C CNN
 F 1 "GND" H 2350 2450 50  0000 C CNN
 F 2 "" H 2350 2600 50  0001 C CNN
@@
 $EndComp
 $Comp
-L +5V #PWR027
+L +5V #PWR27
 U 1 1 5AEDE49D
 P 2050 1950
-F 0 "#PWR027" H 2050 1800 50  0001 C CNN
+F 0 "#PWR27" H 2050 1800 50  0001 C CNN
 F 1 "+5V" H 2050 2090 50  0000 C CNN
 F 2 "" H 2050 1950 50  0001 C CNN
@@
 $EndComp
 $Comp
-L +5V #PWR028
+L +5V #PWR28
 U 1 1 5AEDE4A3
 P 2050 2950
-F 0 "#PWR028" H 2050 2800 50  0001 C CNN
+F 0 "#PWR28" H 2050 2800 50  0001 C CNN
 F 1 "+5V" H 2050 3090 50  0000 C CNN
 F 2 "" H 2050 2950 50  0001 C CNN
