File: power_supply.sch (KiCad schematic (older format))
At the start: 1 part

Commit message: Annotate and add negative IOC faults.
Parts:
- gave numbers to parts that had none: 1
Changed lines of the file:
@@
 $EndDescr
 $Comp
-L Conn_01x03 J?
+L Conn_01x03 J10
 U 1 1 5B013AB0
 P 5150 4100
-F 0 "J?" H 5150 4300 50  0000 C CNN
+F 0 "J10" H 5150 4300 50  0000 C CNN
 F 1 "Conn_01x03" H 5150 3900 50  0000 C CNN
 F 2 "" H 5150 4100 50  0001 C CNN
@@
 $EndComp
 $Comp
-L +24V #PWR?
+L +24V #PWR85
 U 1 1 5B013BF5
 P 5500 3900
-F 0 "#PWR?" H 5500 3750 50  0001 C CNN
+F 0 "#PWR85" H 5500 3750 50  0001 C CNN
 F 1 "+24V" H 5500 4040 50  0000 C CNN
 F 2 "" H 5500 3900 50  0001 C CNN
@@
 $EndComp
 $Comp
-L +5V #PWR?
+L +5V #PWR87
 U 1 1 5B013C0B
 P 5700 3900
-F 0 "#PWR?" H 5700 3750 50  0001 C CNN
+F 0 "#PWR87" H 5700 3750 50  0001 C CNN
 F 1 "+5V" H 5700 4040 50  0000 C CNN
 F 2 "" H 5700 3900 50  0001 C CNN
@@
 $EndComp
 $Comp
-L GND #PWR?
+L GND #PWR86
 U 1 1 5B013C21
 P 5600 4300
-F 0 "#PWR?" H 5600 4050 50  0001 C CNN
+F 0 "#PWR86" H 5600 4050 50  0001 C CNN
 F 1 "GND" H 5600 4150 50  0000 C CNN
 F 2 "" H 5600 4300 50  0001 C CNN
